File: CatEye/Head board/Laser head board.sch (EAGLE design)
At the start: 17 parts, among them X1 DVI-D-R, X2 SMA-R

Commit message: STEP files
Parts:
- C1: device OCR:C3216X7R2E473K160AA -> headboard:OCR_C3216X7R2E473K160AA
- L1: device OCR:SLF7032T -> headboard:OCR_SLF7032T
- LASER: device OCR:CONN_03 -> headboard:OCR_CONN_03
- LD1: device OCR:WP130WCP/2EGW -> headboard:OCR_WP130WCP/2EGW
- PBB150: device OCR:PBB150 -> headboard:OCR_PBB150
- PIEZO, TEC, THERM: device OCR:CONN_02 -> headboard:OCR_CONN_02
- R1, R2, R3, R4, R5, R6: device OCR:RESISTOR -> headboard:OCR_RESISTOR
- X1: device OCR:DVI-D-R_74320 -> headboard:OCR_DVI-D-R_74320
- X2: device OCR:SMA-R/A -> headboard:OCR_SMA-R/A
- ZD: device OCR:MMSZ3V3T1G -> headboard:OCR_MMSZ3V3T1G
Connections:
- net N$7: now also PBB150B.A; no longer PBB150B.C
- net N$8: now also PBB150B.C; no longer PBB150B.A
Other:
- moved on the sheet: PBB150B
