File: CatEye/Head board/Original/Laser head board.brd (EAGLE design)
At the start: 70.3 x 28.4 mm, 18 parts, among them X1 DVI-D-R, X2 SMA-R

Commit message: STEP files
Parts:
- X1: device OCR:DVI-D-R -> headboard:OCR_DVI-D-R
