File: CatEye/Head board/Original/Laser head board.sch (EAGLE design)
At the start: 17 parts, among them X1 DVI-D-R, X2 SMA-R

Commit message: STEP files
Parts:
- X1: device OCR:DVI-D-R_74320 -> headboard:OCR_DVI-D-R_74320
Changed lines of the file:
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@@
 <?xml version="1.0" encoding="utf-8"?>
 <!DOCTYPE eagle SYSTEM "eagle.dtd">
-<eagle version="9.3.0">
+<eagle version="9.6.2">
 <drawing>
 <settings>
@@
 <part name="R4" library="OCR" library_urn="urn:adsk.eagle:library:8062975" deviceset="RESISTOR" device="" package3d_urn="urn:adsk.eagle:package:8116984/2" value="43R"/>
 <part name="PBB150" library="OCR" library_urn="urn:adsk.eagle:library:8062975" deviceset="PBB150" device="" package3d_urn="urn:adsk.eagle:package:8063021/2"/>
-<part name="X1" library="OCR" library_urn="urn:adsk.eagle:library:8062975" deviceset="DVI-D-R" device="_74320" package3d_urn="urn:adsk.eagle:package:8063018/2" value="DVI-D-R"/>
+<part name="X1" library="headboard" library_urn="urn:adsk.eagle:library:49120877" deviceset="OCR_DVI-D-R" device="_74320" package3d_urn="urn:adsk.eagle:package:49120904/1" value="DVI-D-R"/>
 <part name="LD1" library="OCR" library_urn="urn:adsk.eagle:library:8062975" deviceset="WP130WCP/2EGW" device="" package3d_urn="urn:adsk.eagle:package:8063024/2"/>
 <part name="ZD" library="OCR" library_urn="urn:adsk.eagle:library:8062975" deviceset="MMSZ3V3T1G" device="" package3d_urn="urn:adsk.eagle:package:8068621/4" value="3.3V"/>
